File: matek_microbec_6_30v.kicad_pcb (KiCad board)
At the start: 2 copper layers, 14.1 x 9.9 mm, 16 parts, among them U1 MP9943GQ-Z

Commit message: step file
Other:
- board text added: "9V"
Changed lines of the file:
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@@
 		(tags "capacitor")
 		(property "Reference" "C7"
-			(at 1.438888 -0.151391 180)
+			(at 1.338888 -7.951391 180)
 			(layer "F.SilkS")
 			(effects
@@
 		)
 	)
+	(gr_text "9V"
+		(at 135.499762 62.652663 0)
+		(layer "F.SilkS")
+		(effects
+			(font
+				(size 0.5 0.5)
+				(thickness 0.1)
+			)
+			(justify left bottom)
+		)
+	)
